File: MoistureSensor1.kicad_sch (KiCad schematic)
At the start: 38 parts, among them J2 USB C Power Input, J3 SMX Header, J4 Expansion header, J5 Moisture sensors, J6 Power input & Temp sensors, SW1 SW_Slide_DPDT, U1 ESP32-DevKitC, U2 TPS27081ADDCR, U3 TPS27081ADDCR, U4 74HC595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

Commit message: Misc updates
Miscellaneous updates
Parts:
- 5v in1: renamed from J2; value USB C Power Input -> 10164359-00011LF
- C1, C2, C5, C6, C7, C8: footprint Capacitor_THT:C_Axial_L3.8mm_D2.6mm_P5.5mm_Horizontal -> Capacitor_SMD:C_0805_2012Metric_Pad1.18x1.45mm_HandSolder
- H1, H2, H3, H4: footprint MountingHole:MountingHole_3.2mm_M3_ISO7380 -> MountingHole:MountingHole_2.7mm_M2.5_ISO14580
- J1: renamed from J6; value Power input & Temp sensors -> Screw_Terminal_01x08; footprint Ians_Parts:PhoenixContact_MSTBA_2,5_2-G-5,00_1x8_2.50mm_45deg compact -1989803 -> Ians_Parts:PHOENIX_1990067
- J2: renamed from J4; value Expansion header -> Expansion
- J3: renamed from J5; value Moisture sensors -> Screw_Terminal_01x12; footprint Ians_Parts:PhoenixContact_MSTBA_2,5_2-G-5,00_1x12_2.5mm_45deg compact -> Ians_Parts:PHOENIX_1990106
- R1, R2: footprint Resistor_THT:R_Axial_DIN0204_L3.6mm_D1.6mm_P5.08mm_Horizontal -> Resistor_SMD:R_1206_3216Metric_Pad1.30x1.75mm_HandSolder
- R10: renamed from R6; footprint Resistor_SMD:R_1206_3216Metric -> Resistor_SMD:R_1206_3216Metric_Pad1.30x1.75mm_HandSolder
- R11: renamed from R7; footprint Resistor_SMD:R_1206_3216Metric -> Resistor_SMD:R_1206_3216Metric_Pad1.30x1.75mm_HandSolder
- R12: renamed from R8; footprint Resistor_SMD:R_1206_3216Metric -> Resistor_SMD:R_1206_3216Metric_Pad1.30x1.75mm_HandSolder
- R13: renamed from R9; footprint Resistor_THT:R_Axial_DIN0204_L3.6mm_D1.6mm_P5.08mm_Horizontal -> Resistor_SMD:R_1206_3216Metric_Pad1.30x1.75mm_HandSolder
- R3: renamed from R10; footprint Resistor_THT:R_Axial_DIN0204_L3.6mm_D1.6mm_P5.08mm_Horizontal -> Resistor_SMD:R_1206_3216Metric_Pad1.30x1.75mm_HandSolder
- R4: renamed from R11; footprint Resistor_THT:R_Axial_DIN0204_L3.6mm_D1.6mm_P5.08mm_Horizontal -> Resistor_SMD:R_1206_3216Metric_Pad1.30x1.75mm_HandSolder
- R5: renamed from R12; footprint Resistor_SMD:R_1206_3216Metric -> Resistor_SMD:R_1206_3216Metric_Pad1.30x1.75mm_HandSolder
- R6: renamed from R13; footprint Resistor_SMD:R_1206_3216Metric -> Resistor_SMD:R_1206_3216Metric_Pad1.30x1.75mm_HandSolder
- R7: renamed from R3; footprint Resistor_SMD:R_1206_3216Metric -> Resistor_SMD:R_1206_3216Metric_Pad1.30x1.75mm_HandSolder
- R8: renamed from R4; footprint Resistor_SMD:R_1206_3216Metric -> Resistor_SMD:R_1206_3216Metric_Pad1.30x1.75mm_HandSolder
- R9: renamed from R5; footprint Resistor_SMD:R_1206_3216Metric -> Resistor_SMD:R_1206_3216Metric_Pad1.30x1.75mm_HandSolder
- renumbered SW1 to DPDT1, J3 to SMX1
Connections:
- net at R7.1, U5.13, U5.5: now also U4.5 (QF); no longer U4.15 (QA)
- net at R8.1, U5.12, U5.6: now also U4.4 (QE); no longer U4.1 (QB)
- net at R11.1, U7.13, U7.5: now also U4.1 (QB); no longer U4.4 (QE)
- net at R9.1, U6.13, U6.5: now also U4.3 (QD); no longer U4.2 (QC)
- net at R10.1, U6.12, U6.6: now also U4.2 (QC); no longer U4.3 (QD)
- net at R12.1, U7.12, U7.6: now also U4.15 (QA); no longer U4.5 (QF)
