File: MoistureSensor1.kicad_pcb (KiCad board)
At the start: 2 copper layers, 111 x 58 mm, 38 parts, among them J4 Expansion, J5 Screw_Terminal_01x12, J6 Screw_Terminal_01x08, U1 ESP32-DevKitC, U2 TPS27081ADDCR, U3 TPS27081ADDCR, U4 74HC595, U5 CD4066BE, U6 CD4066BE, U7 CD4066BE

Commit message: Misc updates
Miscellaneous updates
Parts:
- added ?: , clipboard:c5f2482b-6cae-4589-8a9f-ca96de6d0741, F.Cu at (214.0, 86.0)
- 5v in1: renamed from 5v in
- DPDT1: renamed from On     Off
- H1, H2, H3, H4: footprint MountingHole:MountingHole_3.2mm_M3_ISO7380 -> MountingHole:MountingHole_2.7mm_M2.5_ISO14580
- J1: renamed from J6; footprint Ians_Parts:PhoenixContact_MSTBA_2,5_2-G-5,00_1x8_2.50mm_45deg compact -1989803 -> Ians_Parts:PHOENIX_1990067
- J3: renamed from J5; footprint Ians_Parts:PhoenixContact_MSTBA_2,5_2-G-5,00_1x12_2.5mm_45deg compact -> Ians_Parts:PHOENIX_1990106
- moved C4 42.4 mm to (203.7, 118.2), turned to 180 degrees
- moved J3 30.6 mm to (97.5, 83.2), turned to -90 degrees
- moved DPDT1 25.0 mm to (198.2, 75.4)
- moved J1 20.8 mm to (165.2, 70.8), turned to 180 degrees
- moved J2 2.94 mm to (202.2, 104.0)
- moved C3 2.76 mm to (203.7, 111.8)
- moved H1 2.12 mm to (204.5, 73.5)
- moved H2 2.12 mm to (204.5, 124.5)
- moved H3 2.12 mm to (100.5, 124.5)
- moved H4 2.12 mm to (100.5, 73.5)
- moved U1 1.00 mm to (194.5, 126.2)
- moved 5v in1 0.60 mm to (115.0, 73.8)
- moved C2 0.25 mm to (136.2, 89.5)
- moved C6 0.25 mm to (140.0, 100.5)
- moved C7 0.10 mm to (140.0, 124.2)
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- renumbered J4 to J2, R6 to R10, R7 to R11, R8 to R12, R9 to R13, R10 to R3, R11 to R4, R12 to R5, R13 to R6, R3 to R7, R4 to R8, R5 to R9, SMX to SMX1
Connections:
- R10 pad 1: Net-(U4-QD) -> Net-(U4-QC)
- R11 pad 1: Net-(U4-QE) -> Net-(U4-QB)
- R12 pad 1: Net-(U4-QF) -> Net-(U4-QA)
- R7 pad 1: Net-(U4-QA) -> Net-(U4-QF)
- R8 pad 1: Net-(U4-QB) -> Net-(U4-QE)
- R9 pad 1: Net-(U4-QC) -> Net-(U4-QD)
- U5 pad 12: Net-(U4-QB) -> Net-(U4-QE)
- U5 pad 13: Net-(U4-QA) -> Net-(U4-QF)
- U5 pad 5: Net-(U4-QA) -> Net-(U4-QF)
- U5 pad 6: Net-(U4-QB) -> Net-(U4-QE)
- U6 pad 12: Net-(U4-QD) -> Net-(U4-QC)
- U6 pad 13: Net-(U4-QC) -> Net-(U4-QD)
- U6 pad 5: Net-(U4-QC) -> Net-(U4-QD)
- U6 pad 6: Net-(U4-QD) -> Net-(U4-QC)
- U7 pad 12: Net-(U4-QF) -> Net-(U4-QA)
- U7 pad 13: Net-(U4-QE) -> Net-(U4-QB)
- U7 pad 5: Net-(U4-QE) -> Net-(U4-QB)
- U7 pad 6: Net-(U4-QF) -> Net-(U4-QA)
Routing:
- net +5VA: track 224.9 -> 255.8 mm
- net Net-(5v in1-GND_A): track 64.8 -> 89.9 mm
- net Net-(5v in1-VBUS_A): track 65.5 -> 90.5 mm
- net Net-(U4-QB): track 60.9 -> 42.8 mm, vias 2 -> 3
- net Net-(U4-QF): track 55.4 -> 37.8 mm, vias 2 -> 3
- net Net-(U4-QA): track 62.4 -> 52.3 mm, vias 5 -> 3
- net Net-(U4-QC): track 35.8 -> 42.2 mm, vias 3 -> 2
- net Net-(U4-QE): track 49.8 -> 43.5 mm, vias 3 -> 2
- net Net-(U3-ON/OFF): track 47.5 -> 52.7 mm
- net Net-(U4-QD): track 42.7 -> 39.3 mm, vias 2 -> 3
- net +3.3VA: track 105.3 -> 107.8 mm
- net Net-(J2-Pin_4): track 8.70 -> 11.1 mm
- net Net-(J2-Pin_3): track 8.70 -> 11.1 mm
- net Net-(J1-Pin_1): track 69.4 -> 67.1 mm
- net Net-(U2-ON/OFF): track 57.6 -> 59.7 mm
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Other:
- outline, holes or cut-outs redrawn
- board text added: "1 0"
- board text removed: "WayWayWay"

Commit message: Small adjustments
Small adjustments
Routing:
- net +5VA: track 255.8 -> 264.4 mm
Changed lines of the file:
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@@
+	)
+	(segment
+		(start 131.5375 89.5)
+		(end 133.374603 91.337103)
+		(width 0.6)
+		(layer "F.Cu")
+		(net 1)
 	)
 	(segment
@@
 		(width 0.6)
 		(layer "F.Cu")
+		(net 1)
+	)
+	(segment
+		(start 133.374603 91.337103)
+		(end 139.374603 91.337103)
+		(width 0.6)
+		(layer "F.Cu")
